Commit message: urdf

File: install/arduinobot_description/share/arduinobot_description/urdf/arduinobot_urdf.xacro (robot description, xacro)
@@ -63,3 +63,47 @@
         <limit lower="-${PI/2}" upper="${PI/2}" effort="${effort}" velocity="${velocity}"/>
     </joint>
+    <link name="claw_support">
+        <visual>
+            <origin rpy="0 0 ${PI/2}" xyz="0 -0.05 -0.15"/>
+            <geometry>
+                <mesh filename="package://arduinobot_description/meshes/claw_support.STL" scale="0.01 0.01 0.01"/>
+            </geometry>
+        </visual>
+    </link>
+    <joint name="horizontal_arm_to_claw_support" type="fixed">
+        <parent link="horizontal_arm"/>
+        <child link="claw_support"/>
+        <origin xyz="0 0.82 0" rpy="0 0 0"/>
+    </joint>
+    <link name="gripper_right">
+        <visual>
+            <origin xyz="-0.1 0.5 -0.1" rpy="0 0 -${PI/2}"/>
+            <geometry>
+                <mesh filename="package://arduinobot_description/meshes/right_finger.STL" scale="0.01 0.01 0.01"/>
+            </geometry>
+        </visual>
+    </link>
+    <link name="gripper_left">
+        <visual>
+            <origin xyz="-0.04 0.5 -0.1" rpy="0 0 -${PI/2}"/>
+            <geometry>
+                <mesh filename="package://arduinobot_description/meshes/left_finger.STL" scale="0.01 0.01 0.01"/>
+            </geometry>
+        </visual>
+    </link>
+    <joint name="joint_4" type="revolute">
+        <parent link="claw_support"/>
+        <child link="gripper_right"/>
+        <axis xyz="0 0 1"/>
+        <origin rpy="0 0 0" xyz="-0.04 0.13 -0.1"/>
+        <limit lower="-${PI/2}" upper="0.0" effort="${effort}" velocity="${velocity}"/>
+    </joint>
+    <joint name="joint_5" type="revolute">
+        <parent link="claw_support"/>
+        <child link="gripper_left"/>
+        <axis xyz="0 0 1"/>
+        <origin rpy="0 0 0" xyz="-0.22 0.13 -0.1"/>
+        <mimic joint="joint_4" multiplier="-1"/>
+        <limit lower="0.0" upper="${PI/2}" effort="${effort}" velocity="${velocity}"/>
+    </joint>
 </robot>

File: src/arduinobot_description/urdf/arduinobot_urdf.xacro (robot description, xacro)
@@ -76,3 +76,34 @@
         <origin xyz="0 0.82 0" rpy="0 0 0"/>
     </joint>
+    <link name="gripper_right">
+        <visual>
+            <origin xyz="-0.1 0.5 -0.1" rpy="0 0 -${PI/2}"/>
+            <geometry>
+                <mesh filename="package://arduinobot_description/meshes/right_finger.STL" scale="0.01 0.01 0.01"/>
+            </geometry>
+        </visual>
+    </link>
+    <link name="gripper_left">
+        <visual>
+            <origin xyz="-0.04 0.5 -0.1" rpy="0 0 -${PI/2}"/>
+            <geometry>
+                <mesh filename="package://arduinobot_description/meshes/left_finger.STL" scale="0.01 0.01 0.01"/>
+            </geometry>
+        </visual>
+    </link>
+    <joint name="joint_4" type="revolute">
+        <parent link="claw_support"/>
+        <child link="gripper_right"/>
+        <axis xyz="0 0 1"/>
+        <origin rpy="0 0 0" xyz="-0.04 0.13 -0.1"/>
+        <limit lower="-${PI/2}" upper="0.0" effort="${effort}" velocity="${velocity}"/>
+    </joint>
+    <joint name="joint_5" type="revolute">
+        <parent link="claw_support"/>
+        <child link="gripper_left"/>
+        <axis xyz="0 0 1"/>
+        <origin rpy="0 0 0" xyz="-0.22 0.13 -0.1"/>
+        <mimic joint="joint_4" multiplier="-1"/>
+        <limit lower="0.0" upper="${PI/2}" effort="${effort}" velocity="${velocity}"/>
+    </joint>
 </robot>
